File: PCB/peripherals.kicad_sch (KiCad schematic)
At the start: 20 parts, among them J1 Conn_01x03_Pin, J10 Conn_01x02_Pin, J2 Conn_01x02_Pin, J3 Conn_01x02_Pin, J4 Conn_01x03_Pin, J5 Conn_01x03_Pin, J6 Conn_01x03_Pin, J7 Conn_01x07_Pin, J8 Conn_01x08_Socket, U2 MPU-6050

Commit message: Start of feedback implementation
Parts:
- added C14: 10uF, Capacitor_SMD:C_1206_3216Metric_Pad1.33x1.80mm_HandSolder, symbol Device:C
- added D10, D11, D12, D13, D5, D6, D7, D8, D9: ESD321, Diode_SMD:D_0402_1005Metric_Pad0.77x0.64mm_HandSolder, symbol Device:D
- R4, R5: value 10kΩ -> 4.7kΩ
Connections:
- net +3V3: now also C14.2, D10.2 (A), D11.2 (A), D12.2 (A), D13.2 (A), D5.2 (A), D6.2 (A), D7.2 (A), D9.2 (A)
- net GND: now also C14.1, D10.1 (K), D11.1 (K), D12.1 (K), D13.1 (K), D5.1 (K), D6.1 (K), D7.1 (K), D8.1 (K), D9.1 (K)
- net MOTOR: now also D8.2 (A)
Other:
- moved on the sheet: H1, H2, J1, J2, J5, J7, J8, R6

Commit message: Implemented all feedback except buck converter
Parts:
- removed C14: 10uF, Capacitor_SMD:C_1206_3216Metric_Pad1.33x1.80mm_HandSolder, symbol Device:C
Connections:
- net +3V3: no longer D5.2 (A), D6.2 (A)
- net FLEX_1: now also D6.2 (A)
- net FLEX_2: now also D5.2 (A)
Other:
- moved on the sheet: D6, J2, J3, R6, R7
